Commit message: 20260626_02-00_forward

File: source/Ranger/Ranger/assets/ranger/urdf/ranger.urdf (robot description, URDF)
Before this commit: robot urdf, 13 links, 12 joints
Links:
- link base_link: mass 35.769 -> 55.0
- link lb_Link: mass 6.04761793125612 -> 5.5
- link lf_Link: mass 6.04761793125612 -> 5.5
- link rb_Link: mass 0 -> 5.5
- link rf_Link: mass 6.04761793125612 -> 5.5
- link w_lb: mass 9.42365069276311 -> 8.0
- link w_lf: mass 9.4237 -> 8.0
- link w_rb: mass 9.42365069276311 -> 8.0
- link w_rf: mass 9.4237 -> 8.0
Joints:
- joint g_lb: limit lower=-1 upper=1 effort=10 velocity=5 -> lower=-0.6 upper=0.6 effort=500 velocity=5
- joint g_lf: limit lower=-1 upper=1 effort=10 velocity=5 -> lower=-0.6 upper=0.6 effort=500 velocity=5
- joint g_rb: limit lower=-1 upper=1 effort=10 velocity=5 -> lower=-0.6 upper=0.6 effort=500 velocity=5
- joint g_rf: limit lower=-1 upper=1 effort=10 velocity=5 -> lower=-0.6 upper=0.6 effort=500 velocity=5
- joint w_lb: origin xyz=-0.38089 0.1 -0.23963 rpy=0 0 0 -> xyz=-0.39572 0.1 -0.21180 rpy=0 0 0
- joint w_lf: origin xyz=0.41801041206503 0.100000000000001 -0.166635216581701 rpy=0 0 0 -> xyz=0.39572 0.1 -0.21180 rpy=0 0 0
- joint w_rb: origin xyz=-0.39963 -0.1 -0.20687 rpy=0 0 0 -> xyz=-0.39572 -0.1 -0.21180 rpy=0 0 0
- joint w_rf: origin xyz=0.38434 -0.1 -0.23406 rpy=0 0 0 -> xyz=0.39572 -0.1 -0.21180 rpy=0 0 0
