Commit message: 20260708_16-37_修改urdf+感知链路

File: source/Ranger/Ranger/assets/ranger/urdf/ranger.urdf (robot description, URDF)
Before this commit: robot urdf, 13 links, 12 joints
Links:
- link base_link: mass 55.0 -> 100.00
- link lb_Link: mass 5.5 -> 5
- link lf_Link: mass 5.5 -> 5
- link rb_Link: mass 5.5 -> 5
- link rf_Link: mass 5.5 -> 5
- link w_lb: mass 8.0 -> 3.0
- link w_lf: mass 8.0 -> 3
- link w_rb: mass 8.0 -> 3
- link w_rf: mass 8.0 -> 3
Joints:
- joint g_lb: limit lower=-0.6 upper=0.6 effort=500 velocity=5 -> lower=-0.35 upper=0.35 effort=500 velocity=5
- joint g_lf: limit lower=-0.6 upper=0.6 effort=500 velocity=5 -> lower=-0.35 upper=0.35 effort=500 velocity=5
- joint g_rb: limit lower=-0.6 upper=0.6 effort=500 velocity=5 -> lower=-0.35 upper=0.35 effort=500 velocity=5
- joint g_rf: limit lower=-0.6 upper=0.6 effort=500 velocity=5 -> lower=-0.35 upper=0.35 effort=500 velocity=5
- joint w_lb: origin xyz=-0.39572 0.1 -0.21180 rpy=0 0 0 -> xyz=-0.38089 0.1 -0.23963 rpy=0 0 0
- joint w_lf: origin xyz=0.39572 0.1 -0.21180 rpy=0 0 0 -> xyz=0.41801041206503 0.100000000000001 -0.166635216581701 rpy=0 0 0
- joint w_rb: origin xyz=-0.39572 -0.1 -0.21180 rpy=0 0 0 -> xyz=-0.39963 -0.1 -0.20687 rpy=0 0 0
- joint w_rf: origin xyz=0.39572 -0.1 -0.21180 rpy=0 0 0 -> xyz=0.38434 -0.1 -0.23406 rpy=0 0 0
