Commit message: 20260714_16-00_修正urdf100mm偏置

File: RANGER/urdf/RANGER.urdf (robot description, URDF)
Before this commit: robot urdf, 13 links, 12 joints
Links:
- link base_link: mass 100.00 -> 100.0
- link lb_Link: mass 5 -> 5.0
- link lf_Link: mass 5 -> 5.0
- link rb_Link: mass 5 -> 5.0
- link rf_Link: mass 5 -> 5.0
- link w_lf: mass 3 -> 3.0
- link w_rb: mass 3 -> 3.0
- link w_rf: mass 3 -> 3.0
Joints:
- joint g_lb: limit lower=-0.35 upper=0.35 effort=500 velocity=5 -> lower=-0.35 upper=0.35 effort=800 velocity=3; origin xyz=-0.1 0.3 -0.28 rpy=0 0 0 -> xyz=-0.1 0.300000000000001 -0.279999999999999 rpy=0 0 0
- joint g_lf: limit lower=-0.35 upper=0.35 effort=500 velocity=5 -> lower=-0.35 upper=0.35 effort=800 velocity=3; origin xyz=0.1 0.3 -0.28 rpy=0 0 0 -> xyz=0.1 0.300000000000001 -0.279999999999999 rpy=0 0 0
- joint g_rb: limit lower=-0.35 upper=0.35 effort=500 velocity=5 -> lower=-0.35 upper=0.35 effort=800 velocity=3; origin xyz=-0.1 -0.3 -0.28 rpy=0 0 0 -> xyz=-0.1 -0.299999999999999 -0.280000000000001 rpy=0 0 0
- joint g_rf: limit lower=-0.35 upper=0.35 effort=500 velocity=5 -> lower=-0.35 upper=0.35 effort=800 velocity=3; origin xyz=0.1 -0.3 -0.28 rpy=0 0 0 -> xyz=0.1 -0.299999999999999 -0.280000000000001 rpy=0 0 0
- joint w_lb: origin xyz=-0.38089 0.1 -0.23963 rpy=0 0 0 -> xyz=-0.389711431702996 0.100000000000001 -0.225000000000001 rpy=0 0 0
- joint w_lf: origin xyz=0.41801041206503 0.100000000000001 -0.166635216581701 rpy=0 0 0 -> xyz=0.389711431702996 0.100000000000001 -0.225000000000002 rpy=0 0 0
- joint w_rb: origin xyz=-0.39963 -0.1 -0.20687 rpy=0 0 0 -> xyz=-0.389711431702996 -0.0999999999999991 -0.225000000000002 rpy=0 0 0
- joint w_rf: origin xyz=0.38434 -0.1 -0.23406 rpy=0 0 0 -> xyz=0.389711431702996 -0.0999999999999991 -0.225000000000002 rpy=0 0 0
